File: pcb/pcbv/pcbv.kicad_sch (KiCad schematic)
At the start: 42 parts, among them J1 Conn_ST_STDC14, J2 I2C, J3 Conn_01x02_Pin, J4 CAN+POWER, J5 CAN, J6 3.3V, J7 5V, SW1 generic 6mm tht switch, U1 MPRLS0025PA00001A, U2 STM32C092RCT6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

Commit message: initial pcb rev
Parts:
- removed J3: Conn_01x02_Pin, Connector_PinHeader_2.54mm:PinHeader_1x02_P2.54mm_Vertical, symbol Connector:Conn_01x02_Pin
- removed SW1: generic 6mm tht switch, Button_Switch_THT:SW_PUSH_6mm, symbol Switch:SW_MEC_5G
- added SW1: generic 6mm tht switch, Button_Switch_THT:SW_PUSH_6mm, symbol Switch:SW_Push
- C1, C11, C7, C8, C9: footprint (none) -> Capacitor_SMD:C_0805_2012Metric
- C10, C12, C13, C14, C15, C16, C17, C2, C3, C4, C5, C6: footprint (none) -> Capacitor_SMD:C_1210_3225Metric
Connections:
- net GND: now also SW1.1
- net CANH: now reaches J4.2 (Pin_2), R5.1, U6.7 (CANH)
- net CANL: now reaches J4.3 (Pin_3), R5.2, U6.6 (CANL)
- net NO+: now reaches C1.1, U1.4 (VO+)
- net NO-: now reaches C1.2, U1.6 (VO-)
- net OSC_OUT: now reaches C8.1, Y1.3
- net OSC_OUT: now also U2.11 (PF1-OSC_OUT)
- net SDA: now reaches J2.1 (Pin_1), R2.1, U2.63 (PB9)
- net SDA: now also U1.2 (MOSI/SDA), U3.10 (SDA)
- net CAN_TX: now reaches U6.1 (TXD)
- net CAN_TX: now also J5.1 (Pin_1), U2.51 (PD1)
- net CAN_RX: now reaches U6.4 (RXD)
- net CAN_RX: now also J5.2 (Pin_2), U2.50 (PD0)
- net OSC_IN: now reaches C7.1, Y1.1
- net OSC_IN: now also U2.10 (PF0-OSC_IN)
- net SCL: now reaches U3.9 (SCL)
- net SCL: now also J2.2 (Pin_2), R1.2, U1.3 (SCLK/SCL), U2.62 (PB8)
- net NRST: now reaches C2.1, D1.1 (K), U2.12 (PF2-NRST)
- net NRST: now also J1.12 (~{RST}), SW1.2
- net OSCX_OUT: now reaches C11.1, Y2.2
- net OSCX_OUT: now also U2.5 (PC15-OSCX_OUT)
- net EOC: now reaches U1.8 (EOC)
- net EOC: now also U2.61 (PB7)
- net RES: now reaches U1.9 (RES)
- net OSCX_IN: now reaches C9.1, Y2.1
- net OSCX_IN: now also U2.4 (PC14-OSCX_IN)
- net VCP_TX: now reaches U2.19 (PA2)
- net VCP_TX: now also J1.14 (VCP_TX)
- net VCP_RX: now reaches U2.20 (PA3)
- net VCP_RX: now also J1.13 (VCP_RX)
- net SWDIO: now reaches U2.45 (PA13)
- net SWDIO: now also J1.4 (JTMS/SWDIO)
- net SWCLK: now reaches U2.46 (PA14-BOOT0)
- net SWCLK: now also J1.6 (JCLK/SWCLK)

Commit message: pcb updated
Parts:
- added F1: Fuse, Fuse:Fuseholder_Clip-5x20mm_Bel_FC-203-22_Lateral_P17.80x5.00mm_D1.17mm_Horizontal, symbol Device:Fuse
- L1: value 18u-RLB0914-180KL -> 18u; footprint Inductor_THT:L_Radial_D8.7mm_P5.00mm_Fastron_07HCP -> Inductor_SMD:L_Taiyo-Yuden_MD-5050
- U4: value LV2862YDDC -> LV2862YDDCT
- U5: value TLV709A50DBZR -> TLV709A50
Connections:
- net VDD: now also F1.1; no longer J4.1 (Pin_1)
- new net: F1.2, J4.1 (Pin_1)
Other:
- moved on the sheet: D1
Changed lines of the file:
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@@
 	)
 	(junction
-		(at 53.34 246.38)
-		(diameter 0)
-		(color 0 0 0 0)
-	)
-	(junction
 		(at 318.77 78.74)
 		(diameter 0)
@@
 	)
 	(junction
+		(at 67.31 246.38)
+		(diameter 0)
+		(color 0 0 0 0)
+	)
+	(junction
 		(at 36.83 33.02)
 		(diameter 0)
@@
 	(wire
 		(pts
-			(xy 53.34 246.38) (xy 53.34 247.65)
+			(xy 67.31 246.38) (xy 67.31 247.65)
 		)
 		(stroke
@@
 	(wire
 		(pts
-			(xy 48.26 256.54) (xy 53.34 256.54)
+			(xy 48.26 256.54) (xy 67.31 256.54)
 		)
 		(stroke
@@
 	(wire
 		(pts
-			(xy 53.34 255.27) (xy 53.34 256.54)
+			(xy 67.31 255.27) (xy 67.31 256.54)
 		)
 		(stroke
@@
 	(wire
 		(pts
+			(xy 359.41 21.59) (xy 365.76 21.59)
+		)
+		(stroke
+			(width 0)
+			(type default)
+		)
+	)
+	(wire
+		(pts
 			(xy 254 45.72) (xy 254 44.45)
 		)
@@
 	(wire
 		(pts
-			(xy 314.96 78.74) (xy 318.77 78.74)
+			(xy 346.71 20.32) (xy 351.79 20.32)
+		)
+		(stroke
+			(width 0)
+			(type default)
+		)
+	)
+	(wire
+		(pts
+			(xy 351.79 20.32) (xy 351.79 21.59)
+		)
+		(stroke
+			(width 0)
+			(type default)
+		)
+	)
+	(wire
+		(pts
+			(xy 297.18 78.74) (xy 318.77 78.74)
 		)
 		(stroke
@@
 	(wire
 		(pts
-			(xy 74.93 77.47) (xy 74.93 80.01)
+			(xy 67.31 246.38) (xy 74.93 246.38)
 		)
 		(stroke
@@
 	(wire
 		(pts
-			(xy 157.48 88.9) (xy 157.48 90.17)
+			(xy 74.93 77.47) (xy 74.93 80.01)
 		)
 		(stroke
@@
 	(wire
 		(pts
-			(xy 87.63 85.09) (xy 91.44 85.09)
+			(xy 157.48 88.9) (xy 157.48 90.17)
 		)
 		(stroke
@@
 	(wire
 		(pts
-			(xy 53.34 246.38) (xy 74.93 246.38)
+			(xy 87.63 85.09) (xy 91.44 85.09)
 		)
 		(stroke
@@
 	(wire
 		(pts
-			(xy 43.18 246.38) (xy 53.34 246.38)
+			(xy 43.18 246.38) (xy 67.31 246.38)
 		)
 		(stroke
@@
 	(wire
 		(pts
-			(xy 365.76 26.67) (xy 365.76 29.21)
+			(xy 365.76 21.59) (xy 365.76 29.21)
 		)
 		(stroke
@@
 	(symbol
 		(lib_id "power:VDD")
-		(at 314.96 78.74 0)
+		(at 297.18 78.74 0)
 		(unit 1)
 		(exclude_from_sim no)
@@
 		(fields_autoplaced yes)
 		(property "Reference" "#PWR026"
-			(at 314.96 82.55 0)
+			(at 297.18 82.55 0)
 			(effects
 				(font
@@
 		)
 		(property "Value" "VDD"
-			(at 314.96 73.66 0)
+			(at 297.18 73.66 0)
 			(effects
 				(font
@@
 		)
 		(property "Footprint" ""
-			(at 314.96 78.74 0)
+			(at 297.18 78.74 0)
 			(effects
 				(font
@@
 		)
 		(property "Datasheet" ""
-			(at 314.96 78.74 0)
+			(at 297.18 78.74 0)
 			(effects
 				(font
@@
 		)
 		(property "Description" "Power symbol creates a global label with name \"VDD\""
-			(at 314.96 78.74 0)
+			(at 297.18 78.74 0)
 			(effects
 				(font
@@
 	(symbol
 		(lib_id "Device:D_Schottky")
-		(at 53.34 251.46 270)
+		(at 67.31 251.46 270)
 		(unit 1)
 		(exclude_from_sim no)
@@
 		(fields_autoplaced yes)
 		(property "Reference" "D1"
-			(at 55.88 249.8724 90)
+			(at 69.85 249.8724 90)
 			(effects
 				(font
@@
 		)
 		(property "Value" "ESDZL5-1F4"
-			(at 55.88 252.4124 90)
+			(at 69.85 252.4124 90)
 			(effects
 				(font
@@
 		)
 		(property "Footprint" "Diode_SMD:D_0201_0603Metric"
-			(at 53.34 251.46 0)
+			(at 67.31 251.46 0)
 			(effects
 				(font
@@
 		)
 		(property "Datasheet" "~"
-			(at 53.34 251.46 0)
+			(at 67.31 251.46 0)
 			(effects
 				(font
@@
 		)
 		(property "Description" "Schottky diode"
-			(at 53.34 251.46 0)
+			(at 67.31 251.46 0)
 			(effects
 				(font
@@
 		)
 		(property "KLC_S3.3" ""
-			(at 53.34 251.46 90)
+			(at 67.31 251.46 90)
 			(effects
 				(font
@@
 		)
 		(property "KLC_S4.1" ""
-			(at 53.34 251.46 90)
+			(at 67.31 251.46 90)
 			(effects
 				(font
@@
 	(symbol
 		(lib_id "power:VDD")
-		(at 365.76 26.67 0)
+		(at 346.71 20.32 0)
 		(unit 1)
 		(exclude_from_sim no)
@@
 		(fields_autoplaced yes)
 		(property "Reference" "#PWR036"
-			(at 365.76 30.48 0)
+			(at 346.71 24.13 0)
 			(effects
 				(font
@@
 		)
 		(property "Value" "VDD"
-			(at 365.76 21.59 0)
+			(at 346.71 15.24 0)
 			(effects
 				(font
@@
 		)
 		(property "Footprint" ""
-			(at 365.76 26.67 0)
+			(at 346.71 20.32 0)
 			(effects
 				(font
@@
 		)
 		(property "Datasheet" ""
-			(at 365.76 26.67 0)
+			(at 346.71 20.32 0)
 			(effects
 				(font
@@
 		)
 		(property "Description" "Power symbol creates a global label with name \"VDD\""
-			(at 365.76 26.67 0)
+			(at 346.71 20.32 0)
 			(effects
 				(font
@@
 			)
 		)
-		(property "Datasheet" "~"
+		(property "Datasheet" "https://www.eaton.com/content/dam/eaton/products/electronic-components/resources/data-sheet/eaton-e9xa-automotive-crystal-resonator-mhz-data-sheet-elx1391-en.pdf"
 			(at 218.44 33.02 0)
 			(effects
@@
 			)
 		)
-		(property "Description" "Four pin crystal, GND on pins 2 and 4"
+		(property "Description" "E9X480072ZA3"
 			(at 218.44 33.02 0)
 			(effects
@@
 			)
 		)
-		(property "Value" "LV2862YDDC"
+		(property "Value" "LV2862YDDCT"
 			(at 248.92 162.56 0)
 			(effects
@@
 			)
 		)
-		(property "Value" "18u-RLB0914-180KL"
+		(property "Value" "18u"
 			(at 293.37 170.18 90)
 			(effects
@@
 			)
 		)
-		(property "Footprint" "Inductor_THT:L_Radial_D8.7mm_P5.00mm_Fastron_07HCP"
+		(property "Footprint" "Inductor_SMD:L_Taiyo-Yuden_MD-5050"
 			(at 293.37 172.72 0)
 			(effects
@@
 			)
 		)
-		(property "Description" "Inductor"
+		(property "Description" "SRN5020TA-180M"
 			(at 293.37 172.72 0)
 			(effects
@@
 			)
 		)
-		(property "Value" "TLV709A50DBZR"
+		(property "Value" "TLV709A50"
 			(at 339.09 101.5999 90)
 			(effects
@@
 			)
 		)
-		(property "Datasheet" "~"
+		(property "Datasheet" "https://www.eaton.com/content/dam/eaton/products/electronic-components/resources/data-sheet/eaton-e3k-crystal-resonator-khz-data-sheet-elx1445-en.pdf"
 			(at 260.35 31.75 0)
 			(effects
@@
 			)
 		)
-		(property "Description" "Two pin crystal"
+		(property "Description" "E3K327071405"
 			(at 260.35 31.75 0)
 			(effects
@@
 					(unit 1)
 				)
+			)
+		)
+	)
+	(symbol
+		(lib_id "Device:Fuse")
+		(at 355.6 21.59 90)
+		(unit 1)
+		(exclude_from_sim no)
+		(in_bom yes)
+		(on_board yes)
+		(dnp no)
+		(fields_autoplaced yes)
+		(property "Reference" "F1"
+			(at 355.6 15.24 90)
+			(effects
+				(font
+					(size 1.27 1.27)
+				)
+			)
+		)
+		(property "Value" "Fuse"
+			(at 355.6 17.78 90)
+			(effects
+				(font
+					(size 1.27 1.27)
+				)
+			)
+		)
+		(property "Footprint" "Fuse:Fuseholder_Clip-5x20mm_Bel_FC-203-22_Lateral_P17.80x5.00mm_D1.17mm_Horizontal"
+			(at 355.6 23.368 90)
+			(effects
+				(font
+					(size 1.27 1.27)
+				)
+				(hide yes)
+			)
+		)
+		(property "Datasheet" "~"
+			(at 355.6 21.59 0)
+			(effects
+				(font
+					(size 1.27 1.27)
+				)
+				(hide yes)
+			)
+		)
+		(property "Description" "Fuse"
+			(at 355.6 21.59 0)
+			(effects
+				(font
+					(size 1.27 1.27)
+				)
+				(hide yes)
+			)
+		)
+		(pin "1"
+		)
+		(pin "2"
+		)
+		(instances
+			(project "pcbv"
+				(path "/96fbe704-c415-4a54-ac40-dd09e6fa9554"
+					(reference "F1")
+					(unit 1)
+				)
